Commit message: add offset to driver

File: cobot_v06_ep02/robots/cobot_v06_ep02.urdf (robot description, URDF)
Before this commit: robot cobot_v06_ep02, 8 links, 7 joints
Joints:
- joint J_tool: origin xyz=0 0 0.01036 rpy=0 0 0 -> xyz=0 0 0.05 rpy=0 0 0

Commit message: before intgrate

File: cobot_v06_ep02/robots/cobot_v06_ep02.urdf (robot description, URDF)
Before this commit: robot cobot_v06_ep02, 8 links, 7 joints
Joints:
- joint J1: limit lower=-1.5 upper=1.5 effort=0 velocity=0 -> lower=-2.36 upper=2.36 effort=0 velocity=0
- joint J_tool: origin xyz=0 0 0.05 rpy=0 0 0 -> xyz=0 0 0.081 rpy=0 0 0

Commit message: text to point

File: cobot_v06_ep02/robots/cobot_v06_ep02.urdf (robot description, URDF)
Before this commit: robot cobot_v06_ep02, 8 links, 7 joints
Joints:
- joint J2: limit lower=-1.2214 upper=2.25 effort=0 velocity=0 -> lower=-1.05 upper=0.52 effort=0 velocity=0
- joint J3: limit lower=-3.45 upper=1.25 effort=0 velocity=0 -> lower=-2.36 upper=0.79 effort=0 velocity=0
- joint J4: limit lower=-3.15 upper=3.15 effort=0 velocity=0 -> lower=-2.36 upper=2.36 effort=0 velocity=0
- joint J5: limit lower=-3.15 upper=0.35 effort=0 velocity=0 -> lower=-3.59 upper=0.4499999864 effort=0 velocity=0
- joint J6: limit lower=-3.15 upper=3.15 effort=0 velocity=0 -> effort=0 velocity=0

Commit message: full v1

File: cobot_v06_ep02/robots/cobot_v06_ep02.urdf (robot description, URDF)
Before this commit: robot cobot_v06_ep02, 8 links, 7 joints
Joints:
- joint J6: type revolute -> continuous

Commit message: abc

File: cobot_v06_ep02/robots/cobot_v06_ep02.urdf (robot description, URDF)
Before this commit: robot cobot_v06_ep02, 8 links, 7 joints
Joints:
- joint J2: limit lower=-1.05 upper=0.52 effort=0 velocity=0 -> lower=-1.05 upper=1.0 effort=0 velocity=0
- joint J3: limit lower=-2.36 upper=0.79 effort=0 velocity=0 -> lower=-2.36 upper=1.08 effort=0 velocity=0
- joint J4: limit lower=-2.36 upper=2.36 effort=0 velocity=0 -> lower=-2.87979 upper=2.87979 effort=0 velocity=0

Commit message: abc

File: cobot_v06_ep02/robots/cobot_v06_ep02.urdf (robot description, URDF)
Before this commit: robot cobot_v06_ep02, 8 links, 7 joints
Joints:
- joint J_tool: origin xyz=0 0 0.081 rpy=0 0 0 -> xyz=0 0 0.05 rpy=0 0 0

Commit message: ...

File: cobot_v06_ep02/robots/cobot_v06_ep02.urdf (robot description, URDF)
Before this commit: robot cobot_v06_ep02, 8 links, 7 joints
Joints:
- joint J_tool: origin xyz=0 0 0.05 rpy=0 0 0 -> xyz=0 0 0.081 rpy=0 0 0
